Commit message: Hacks to display angles in debug info. Added example_sliders.py

File: urdf/spotmicroai.urdf.xacro (robot description, xacro)
@@ -178,5 +178,5 @@
       <visual>
         <geometry>
-        <mesh filename="../STL/files/foot.stl" scale="0.001 0.001 0.001"/>
+        <mesh filename="../urdf/stl/foot.stl" scale="0.001 0.001 0.001"/>
         </geometry>
         <origin rpy="0 -0.40010 0" xyz="0 -0.01 0"/>
@@ -237,5 +237,5 @@
     <visual>
       <geometry>
-        <mesh filename="../STL/lidar/rplidar_main.STL" scale="0.001 0.001 0.001"/>
+        <mesh filename="../urdf/stl/rplidar_main.STL" scale="0.001 0.001 0.001"/>
       </geometry>
       <material name="black"/>
